Commit message: adding validity checking for gps

File: launch/ss.urdf (robot description, URDF)
Before this commit: robot streetsmarts, 3 links, 2 joints
Links:
- added link fix_link; visual box size=0.06 0.04 0.02
Joints:
- added joint fix_link_joint: type fixed, parent base_link, child fix_link, origin xyz=0 0 0 rpy=3.1416 0 0

Commit message: working with no fix

File: launch/ss.urdf (robot description, URDF)
Before this commit: robot streetsmarts, 4 links, 3 joints
Links:
- removed link fix_link
Joints:
- removed joint fix_link_joint
- joint camera_link_joint: origin xyz=0.01 0. 0.19 rpy=0. -0.1745 3.1416 -> xyz=-0.8 0. -0.3 rpy=0. 0. 0.; parent imu_link -> base_link
- joint imu_link_joint: origin xyz=0 0 0 rpy=3.1416 0 0 -> xyz=0.0 0 0.0 rpy=0 0 0

Commit message: moving to its own dir, adding new lib

File: launch/ss.urdf (robot description, URDF)
Before this commit: robot streetsmarts, 4 links, 3 joints
Joints:
- joint camera_link_joint: origin xyz=0.01 0. 0.19 rpy=0. -0.1745 3.1416 -> xyz=-0.8 0. 0.3 rpy=0. 0. 0.; parent imu_link -> base_link
- joint fix_link_joint: origin xyz=0 0 0 rpy=3.1416 0 0 -> xyz=0 0 0 rpy=0 0 0
- joint imu_link_joint: origin xyz=0 0 0 rpy=3.1416 0 0 -> xyz=0 0 0 rpy=0 0 0

Commit message: asdfasdf

File: launch/ss.urdf (robot description, URDF)
Before this commit: robot streetsmarts, 4 links, 3 joints
Joints:
- joint camera_link_joint: origin xyz=-0.8 0. 0.3 rpy=0. 0. 0. -> xyz=0. 0. 0. rpy=0. 0. 0.

Commit message: adding correct roll and yaw offsets

File: launch/ss.urdf (robot description, URDF)
Before this commit: robot streetsmarts, 4 links, 3 joints
Joints:
- joint camera_link_joint: origin xyz=0. 0. 0. rpy=0. 0. 0. -> xyz=0. 0. 0.01 rpy=1.57 0. 1.57

Commit message: idk

File: launch/ss.urdf (robot description, URDF)
Before this commit: robot streetsmarts, 4 links, 3 joints
Joints:
- joint camera_link_joint: origin xyz=0. 0. 0.01 rpy=1.57 0. 1.57 -> xyz=0. 0. 0.01 rpy=-1.57 0. -1.57
